Commit message: std

File: config/open_manipulator_x.ros2_control.xacro (robot description, xacro)
@@ -1,60 +1,60 @@
 <?xml version="1.0"?>
 <robot xmlns:xacro="http://www.ros.org/wiki/xacro">
-    <xacro:macro name="open_manipulator_x_ros2_control" params="name initial_positions_file">
-        <xacro:property name="initial_positions" value="${load_yaml(initial_positions_file)['initial_positions']}"/>
-        <ros2_control name="${name}" type="system">
-            <hardware>
-                <plugin>moveit_open_manipulator_x/RobotSystem</plugin>
-            </hardware>
-            <joint name="joint1">
-                <command_interface name="position"/>
-                <state_interface name="position">
-                  <param name="initial_value">${initial_positions['joint1']}</param>
-                </state_interface>
-                <state_interface name="velocity"/>
-            </joint>
-            <joint name="joint2">
-                <command_interface name="position"/>
-                <state_interface name="position">
-                  <param name="initial_value">${initial_positions['joint2']}</param>
-                </state_interface>
-                <state_interface name="velocity"/>
-            </joint>
-            <joint name="joint3">
-                <command_interface name="position"/>
-                <state_interface name="position">
-                  <param name="initial_value">${initial_positions['joint3']}</param>
-                </state_interface>
-                <state_interface name="velocity"/>
-            </joint>
-            <joint name="joint4">
-                <command_interface name="position"/>
-                <state_interface name="position">
-                  <param name="initial_value">${initial_positions['joint4']}</param>
-                </state_interface>
-                <state_interface name="velocity"/>
-            </joint>
-            <joint name="virtual_roll_joint">
-                <command_interface name="position"/>
-                <state_interface name="position">
-                  <param name="initial_value">${initial_positions['virtual_roll_joint']}</param>
-                </state_interface>
-                <state_interface name="velocity"/>
-            </joint>
-            <joint name="virtual_yaw_joint">
-                <command_interface name="position"/>
-                <state_interface name="position">
-                  <param name="initial_value">${initial_positions['virtual_yaw_joint']}</param>
-                </state_interface>
-                <state_interface name="velocity"/>
-            </joint>
-            <joint name="gripper">
-                <command_interface name="position"/>
-                <state_interface name="position">
-                  <param name="initial_value">${initial_positions['gripper']}</param>
-                </state_interface>
-                <state_interface name="velocity"/>
-            </joint>
-        </ros2_control>
-    </xacro:macro>
+  <xacro:macro name="open_manipulator_x_ros2_control" params="name initial_positions_file">
+    <xacro:property name="initial_positions" value="${load_yaml(initial_positions_file)['initial_positions']}"/>
+    <ros2_control name="${name}" type="system">
+      <hardware>
+        <plugin>moveit_open_manipulator_x/RobotSystem</plugin>
+      </hardware>
+      <joint name="joint1">
+        <command_interface name="position"/>
+        <state_interface name="position">
+          <param name="initial_value">${initial_positions['joint1']}</param>
+        </state_interface>
+        <state_interface name="velocity"/>
+      </joint>
+      <joint name="joint2">
+        <command_interface name="position"/>
+        <state_interface name="position">
+          <param name="initial_value">${initial_positions['joint2']}</param>
+        </state_interface>
+        <state_interface name="velocity"/>
+      </joint>
+      <joint name="joint3">
+        <command_interface name="position"/>
+        <state_interface name="position">
+          <param name="initial_value">${initial_positions['joint3']}</param>
+        </state_interface>
+        <state_interface name="velocity"/>
+      </joint>
+      <joint name="joint4">
+        <command_interface name="position"/>
+        <state_interface name="position">
+          <param name="initial_value">${initial_positions['joint4']}</param>
+        </state_interface>
+        <state_interface name="velocity"/>
+      </joint>
+      <joint name="virtual_roll_joint">
+        <command_interface name="position"/>
+        <state_interface name="position">
+          <param name="initial_value">${initial_positions['virtual_roll_joint']}</param>
+        </state_interface>
+        <state_interface name="velocity"/>
+      </joint>
+      <joint name="virtual_yaw_joint">
+        <command_interface name="position"/>
+        <state_interface name="position">
+          <param name="initial_value">${initial_positions['virtual_yaw_joint']}</param>
+        </state_interface>
+        <state_interface name="velocity"/>
+      </joint>
+      <joint name="gripper">
+        <command_interface name="position"/>
+        <state_interface name="position">
+          <param name="initial_value">${initial_positions['gripper']}</param>
+        </state_interface>
+        <state_interface name="velocity"/>
+      </joint>
+    </ros2_control>
+  </xacro:macro>
 </robot>

Commit message: arg

File: config/open_manipulator_x.ros2_control.xacro (robot description, xacro)
@@ -1,9 +1,12 @@
 <?xml version="1.0"?>
 <robot xmlns:xacro="http://www.ros.org/wiki/xacro">
-  <xacro:macro name="open_manipulator_x_ros2_control" params="name initial_positions_file">
-    <xacro:property name="initial_positions" value="${load_yaml(initial_positions_file)['initial_positions']}"/>
+  <xacro:macro name="open_manipulator_x_ros2_control" params="name initial_positions_file usb_port baud_rate">
+    <!-- <xacro:property name="usb_port" value="$(arg usb_port)" default="/dev/ttyUSB0"/> -->
+    <xacro:property name="initial_positions" value="${xacro.load_yaml(initial_positions_file)['initial_positions']}"/>
     <ros2_control name="${name}" type="system">
       <hardware>
         <plugin>moveit_open_manipulator_x/RobotSystem</plugin>
+        <param name="usb_port">${usb_port}</param>
+        <param name="baud_rate">${baud_rate}</param>
       </hardware>
       <joint name="joint1">

File: config/open_manipulator_x.urdf.xacro (robot description, xacro)
@@ -6,4 +6,6 @@
     <!-- Import control_xacro -->
     <xacro:include filename="open_manipulator_x.ros2_control.xacro" />
-    <xacro:open_manipulator_x_ros2_control name="omx" initial_positions_file="$(arg initial_positions_file)"/>
+    <xacro:arg name="usb_port" default="/dev/ttyUSB0" />
+    <xacro:arg name="baud_rate" default="0" />
+    <xacro:open_manipulator_x_ros2_control name="omx" initial_positions_file="$(arg initial_positions_file)" usb_port="$(arg usb_port)" baud_rate="$(arg baud_rate)"/>
 </robot>

Commit message: arg

File: config/open_manipulator_x.ros2_control.xacro (robot description, xacro)
@@ -1,5 +1,5 @@
 <?xml version="1.0"?>
 <robot xmlns:xacro="http://www.ros.org/wiki/xacro">
-  <xacro:macro name="open_manipulator_x_ros2_control" params="name initial_positions_file usb_port baud_rate">
+  <xacro:macro name="open_manipulator_x_ros2_control" params="name initial_positions_file usb_port baud_rate yaml_file interface">
     <!-- <xacro:property name="usb_port" value="$(arg usb_port)" default="/dev/ttyUSB0"/> -->
     <xacro:property name="initial_positions" value="${xacro.load_yaml(initial_positions_file)['initial_positions']}"/>
@@ -9,4 +9,6 @@
         <param name="usb_port">${usb_port}</param>
         <param name="baud_rate">${baud_rate}</param>
+        <param name="yaml_file">${yaml_file}</param>
+        <param name="interface">${interface}</param>
       </hardware>
       <joint name="joint1">

File: config/open_manipulator_x.urdf.xacro (robot description, xacro)
@@ -1,11 +1,20 @@
 <?xml version="1.0"?>
 <robot xmlns:xacro="http://www.ros.org/wiki/xacro" name="open_manipulator_x">
-    <xacro:arg name="initial_positions_file" default="initial_positions.yaml" />
-    <!-- Import open_manipulator_x urdf file -->
-    <xacro:include filename="$(find open_manipulator_x_description)/urdf/open_manipulator_x.urdf.xacro" />
-    <!-- Import control_xacro -->
-    <xacro:include filename="open_manipulator_x.ros2_control.xacro" />
-    <xacro:arg name="usb_port" default="/dev/ttyUSB0" />
-    <xacro:arg name="baud_rate" default="0" />
-    <xacro:open_manipulator_x_ros2_control name="omx" initial_positions_file="$(arg initial_positions_file)" usb_port="$(arg usb_port)" baud_rate="$(arg baud_rate)"/>
+  <xacro:arg name="initial_positions_file" default="initial_positions.yaml" />
+  <!-- Import open_manipulator_x urdf file -->
+  <xacro:include filename="$(find open_manipulator_x_description)/urdf/open_manipulator_x.urdf.xacro" />
+  <!-- Import control_xacro -->
+  <xacro:include filename="open_manipulator_x.ros2_control.xacro" />
+  <xacro:arg name="usb_port" default="/dev/ttyUSB0" />
+  <xacro:arg name="baud_rate" default="1000000" />
+  <xacro:arg name="yaml_file" default="" />
+  <xacro:arg name="interface" default="position" />
+  <xacro:open_manipulator_x_ros2_control
+    name="omx"
+    initial_positions_file="$(arg initial_positions_file)"
+    usb_port="$(arg usb_port)"
+    baud_rate="$(arg baud_rate)"
+    yaml_file="$(arg yaml_file)"
+    interface="$(arg interface)"
+  />
 </robot>
